Commit message: fix(params): adopt Rm=0.593 ohm and mass=0.037 kg ecosystem-wide
Applies the user decision resolving the two UNRESOLVED parameter groups
found by sf params check.

Changes:
- Rm 0.593 ohm (paper LCR measurement, adopted by user decision in commit
  9a656a9f 2026-07-15): genesis motor_model.py (was 0.34), vpython
  motors.py (was 0.63), SIL plant.hpp motor_Rm (was 0.34), sysid
  inertia.py (now sourced from get_flat_defaults, dead-code constants
  de-duplicated), docs tables
- plant.hpp motor_Km 6.12e-4 -> 5.682e-4 (direct measurement 2026-07-16;
  old value was a stale reference calc from legacy Cq*0.34)
- mass 0.037 kg (measured 36.8g; firmware had it since commit 43841314
  2026-03-31): tools/sysid/defaults.py + function defaults in
  motor/drag/validation/sysid CLI, stampfly_edu fallbacks x3, vpython
  run_sim.py, genesis demo, URDFs (base 0.033 + 4x1g props = 0.037) and
  their generator script, simulator/README.md examples
- params_manifest.py: Rm/mass groups flipped from Unresolved to expected
  values (0.593 / 0.037, URDF base 0.033), URDF rows added
- docs: "3-value Rm parallel" note replaced with the resolution (old 0.34 =
  possibly-different-unit LCR, 0.63 = vpython stale init — update gaps, not
  competing measurements); Km adopted=5.682e-4 with formula value 4.51e-4
  noted as an unexplained 20.6% discrepancy; Dm computed value added

Safety evidence:
- genesis/vpython motor ODEs derive Km/Dm/Qf from Rm (Cq*Rm/Am etc.), and
  Rm cancels algebraically from the steady-state equations — hover omega
  and voltage verified numerically bit-identical before/after
- plant.hpp Rm/Km feed only the battery-current estimate (verified in
  plant.cpp; solveOmega uses Am/Bm/Cm only) — outside the deferred
  backlog #3 Ct set
- Verified: sf params check --strict exit 0 (OK=49 MISMATCH=0 UNRESOLVED=0
  EXEMPT=1 ERROR=0), validate_params no warnings, sf sil regression 33/33
  PASS (rerun by reviewer)

Known remaining gap: model omega at hover voltage (~2681 rad/s at 2.1V) vs
measured 3670 rad/s persists — tied to the deferred Ct/Am 3-point
recalibration (backlog #3), unchanged by this commit.

Next steps:
- Investigate the Km formula-vs-measurement 20.6% discrepancy noted in
  stampfly-parameters.md
- Wire sf params check --strict into CI / sf sil regression
- Phase 1: spec YAML + codegen for these parameters (decision pending)

Co-Authored-By: Claude Fable 5 <noreply@anthropic.com>

File: simulator/shared/assets/meshes/parts/stampfly.urdf (robot description, URDF)
Before this commit: robot stampfly, 5 links, 4 joints
Links:
- link base_link: mass 0.030 -> 0.033

File: simulator/shared/assets/meshes/parts/stampfly_fixed.urdf (robot description, URDF)
Before this commit: robot stampfly_fixed, 1 links, 0 joints
Links:
- link base_link: mass 0.035 -> 0.037
